File: Schematics/motor-driver/motor-driver.sch (KiCad schematic (older format))
At the start: 16 parts, among them J1 Conn_01x02_Male, U1 encoder-motor, U2 encoder-motor, U3 encoder-motor, U4 encoder-motor, U5 TB6612-breakout, U6 TB6612-breakout, U8 Teensy4.0

Commit message: Update schematic and start on PCB layout
Parts:
- removed C1, C2: 0.1uF, Capacitors_THT:C_Disc_D5.0mm_W2.5mm_P5.00mm, symbol Device:CP
- removed C3: 10uF, Capacitors_THT:CP_Radial_D10.0mm_P7.50mm, symbol Device:CP
- removed J1: Conn_01x02_Male, Rover:AMASS_XT60-M_1x02_P7.20mm_Vertical, symbol Connector:Conn_01x02_Male
- removed J?: SPI, symbol Connector:Conn_01x07_Female
- removed J?: I2C/Ain/PWM, symbol Connector:Conn_01x05_Female
- removed J?: UART/Ain, symbol Connector:Conn_01x05_Female
- removed J?: UART/I2C/PWM, symbol Connector:Conn_01x05_Female
- removed U1, U2, U3, U4: encoder-motor, Rover:Motor_Header_Pitch2.54mm, symbol rover:encoder-motor
- removed U5, U6: TB6612-breakout, Rover:TB661_breakout, symbol rover:TB6612-breakout
- added 47k1: R, Resistors_SMD:R_0805_HandSoldering, symbol Device:R
- added C1, C2: 10uF, Capacitors_SMD:C_1206_HandSoldering, symbol Device:C
- added C10, C3, C4, C5, C6, C7, C8, C9: 0.1uF, Capacitors_SMD:C_1206_HandSoldering, symbol Device:C
- added J1: XT-60, Rover:AMASS_XT60-M_1x02_P7.20mm_Vertical, symbol rover:XT-60
- added J10: I2C/Ain/PWM 5V, Rover:I2C_Ain_PWM_5V, symbol Connector:Conn_01x04_Female
- added J2: SPI, Rover:SPI_3.3V, symbol Connector:Conn_01x06_Female
- added J3: 32-33, Rover:32-33_3.3V, symbol Connector:Conn_01x02_Female
- added J4: UART/I2C/PWM 3.3V, Rover:UART_I2C_PWM_3.3V, symbol Connector:Conn_01x04_Female
- added J5: I2C/Ain/PWM 3.3V, Rover:I2C_Ain_PWM_3.3V, symbol Connector:Conn_01x04_Female
- added J6: PWM/PPM 3.3V, Rover:PPM_PWM_3.3V, symbol Connector:Conn_01x03_Female
- added J7: UART/Ain, Rover:UART_Ain_3.3V, symbol Connector:Conn_01x04_Female
- added J8: 32-33, Rover:32-33_5V, symbol Connector:Conn_01x02_Female
- added J9: UART/I2C/PWM 5V, Rover:I2C_Ain_PWM_5V, symbol Connector:Conn_01x04_Female
- added M1, M2, M3, M4: encoder-motor, Rover:Motor_Header_Pitch2.54mm, symbol rover:encoder-motor
- added R1: 47k, Resistors_SMD:R_0805_HandSoldering, symbol Device:R
- added U1, U2: TB6612FNG, Housings_SSOP:SSOP-24_5.3x8.2mm_Pitch0.65mm, symbol Driver_Motor:TB6612FNG
- added U3, U4: TXB0108PWR, TXB0108PWR:TSSOP20, symbol TXB0108PWR:TXB0108PWR
- J11: renamed from J?; value PWM/PPM RX -> PWM/PPM 5V; footprint (none) -> Rover:PPM_PWM_5V
- renumbered U8 to U5
Connections:
- net +3V3: now also 47k1.1, C3.2, C6.2, C7.2, C9.2, J2.2 (Pin_2), J5.2 (Pin_2), J7.2 (Pin_2), R1.1, U1.20 (VCC), U2.20 (VCC), U3.10 (OE), U3.2 (VCCA), U4.10 (OE), U4.2 (VCCA)
- net +5V: now also C5.1, C8.1, J10.2 (Pin_2), J4.3 (Pin_3), J6.2 (Pin_2), J9.3 (Pin_3), M1.2 (VCC), M2.2 (VCC), M3.2 (VCC), M4.2 (VCC), U3.19 (VCCB), U4.19 (VCCB)
- net +BATT: now also C1.2, C10.2, C2.2, C4.2, J1.2 (+), U1.13 (VM2), U1.14 (VM3), U1.24 (VM1), U2.13 (VM2), U2.14 (VM3), U2.24 (VM1)
- net -BATT: now also C1.1, C10.1, C2.1, C4.1, J1.1 (-), U1.10 (PGND2), U1.3 (PGND1), U1.4 (PGND1), U1.9 (PGND2), U2.10 (PGND2), U2.3 (PGND1), U2.4 (PGND1), U2.9 (PGND2)
- net GND: now also U5.32 (GND), 47k1.2, C3.1, C5.2, C6.1, C7.1, C8.2, C9.1, J10.1 (Pin_1), J2.1 (Pin_1), J4.4 (Pin_4), J5.1 (Pin_1), J6.1 (Pin_1), J7.1 (Pin_1), J9.4 (Pin_4), M1.5 (GND), M2.5 (GND), M3.5 (GND), M4.5 (GND), R1.2, U1.18 (GND), U2.18 (GND), U3.11 (GND), U4.11 (GND)
- net M1+: now also M1.6 (M+), U1.5 (AO2), U1.6 (AO2)
- net M1-: now also M1.1 (M-), U1.1 (AO1), U1.2 (AO1)
- net M2+: now also M2.6 (M+), U1.7 (BO2), U1.8 (BO2)
- net M2-: now also M2.1 (M-), U1.11 (BO1), U1.12 (BO1)
- net M3+: now also M3.6 (M+), U2.5 (AO2), U2.6 (AO2)
- net M3-: now also M3.1 (M-), U2.1 (AO1), U2.2 (AO1)
- net M4+: now also M4.6 (M+), U2.7 (BO2), U2.8 (BO2)
- net M4-: now also M4.1 (M-), U2.11 (BO1), U2.12 (BO1)
- net STBY: now also U5.42 (31_CTX3), U1.19 (STBY), U2.19 (STBY); no longer U5.10 (8_TX2_IN1)
- net at U5.30 (23_A9_CRX1_MCLK1): now also U2.15 (PWMB)
- net at U5.40 (29_TX7): now also U2.16 (BIN2)
- net at U5.39 (28_RX7): now also U2.17 (BIN1)
- net at U5.37 (26_A12_MOSI1): now also U2.21 (AIN1)
- net at U5.38 (27_A13_SCK1): now also U2.22 (AIN2)
- net at U5.29 (22_A8_CTX1): now also U2.23 (PWMA)
- net at U5.41 (30_CRX3): now also U4.4 (A3)
- net at U5.9 (7_RX2_OUT1A): now also U3.3 (A2)
- net at U5.7 (5_IN2): now also U3.4 (A3)
- net at U5.6 (4_BCLK2): now also U3.5 (A4)
- net at U5.24 (17_A3_TX4_SDA1): now also U1.16 (BIN2)
- net at U5.23 (16_A2_RX4_SCL1): now also U1.17 (BIN1)
- net at U5.21 (14_A0_TX3_SPDIF_OUT): now also U1.21 (AIN1)
- net at U5.22 (15_A1_RX3_SPDIF_IN): now also U1.22 (AIN2)
- net at U5.11 (9_OUT1C): now also U1.15 (PWMB)
- net at U5.5 (3_LRCLK2): now also U3.6 (A5)
- net at U5.4 (2_OUT2): now also U3.7 (A6)
- net at U5.3 (1_TX1_CTX2_MISO1): now also U3.8 (A7)
- net at U5.2 (0_RX1_CRX2_CS1): now also U3.9 (A8)
- net at U5.12 (10_CS_MQSR): now also J2.6 (Pin_6)
- net at U5.13 (11_MOSI_CTX1): now also J2.5 (Pin_5)
- net at U5.14 (12_MISO_MQSL): now also J2.4 (Pin_4)
- net at U5.20 (13_SCK_CRX1_LED): now also J2.3 (Pin_3)
- net at U5.25 (18_A4_SDA0): now also J5.3 (Pin_3), U4.7 (A6)
- net at U5.26 (19_A5_SCL0): now also J5.4 (Pin_4), U4.8 (A7)
- net at U5.27 (20_A6_TX5_LRCLK1): now also J7.3 (Pin_3)
- net at U5.28 (21_A7_RX5_BCLK1): now also J7.4 (Pin_4)
- net at U5.35 (24_A10_TX6_SCL2): now also J4.2 (Pin_2), U4.6 (A5)
- net at U5.36 (25_A11_RX6_SDA2): now also J4.1 (Pin_1), U4.5 (A4)
- net at U5.43 (32_OUT1B): now also J3.2 (Pin_2), U4.3 (A2)
- net at U5.44 (33_MCLK2): now also J3.1 (Pin_1), U4.1 (A1)
- net at U5.8 (6_OUT1D): now also J6.3 (Pin_3), U4.9 (A8); no longer J11.3 (Pin_3)
- new net: U1.23 (PWMA), U5.10 (8_TX2_IN1)
- new net: J10.3 (Pin_3), U4.14 (B6)
- new net: J10.4 (Pin_4), U4.13 (B7)
- new net: M1.4 (A), U3.12 (B8)
- new net: M1.3 (B), U3.13 (B7)
- new net: M2.4 (A), U3.14 (B6)
- new net: M2.3 (B), U3.15 (B5)
- new net: M3.4 (A), U3.16 (B4)
- new net: M3.3 (B), U3.17 (B3)
- new net: M4.4 (A), U3.18 (B2)
- new net: J11.3 (Pin_3), U4.12 (B8)
- new net: M4.3 (B), U4.17 (B3)
- new net: J8.1 (Pin_1), U4.20 (B1)
- new net: J8.2 (Pin_2), U4.18 (B2)
- new net: J9.2 (Pin_2), U4.15 (B5)
- new net: J9.1 (Pin_1), U4.16 (B4)
- no-connect marks 0 -> 18
Other:
- moved on the sheet: J11, U5

Commit message: Finish updating motor driver PCB for Teensy 4.0
Parts:
- removed U3, U4: TXB0108PWR, TXB0108PWR:TSSOP20, symbol TXB0108PWR:TXB0108PWR
- added U3, U4: TXS0108EPW, Housings_SSOP:TSSOP-20_4.4x6.5mm_Pitch0.65mm, symbol Logic_LevelTranslator:TXS0108EPW
- J3: value 32-33 -> 32-33 3.3V
- J8: value 32-33 -> 32-33 5V
- J9: footprint Rover:I2C_Ain_PWM_5V -> Rover:UART_I2C_PWM_5V
- R1: renamed from 47k1; value R -> 47k
- renumbered R1 to R2
Connections:
- net +3V3: now also J4.2 (Pin_2), J6.2 (Pin_2), U3.10 (OE), U3.2 (VCCA), U4.10 (OE), U4.2 (VCCA)
- net +5V: now also J9.2 (Pin_2), U3.19 (VCCB), U4.19 (VCCB); no longer J4.3 (Pin_3), J6.2 (Pin_2), J9.3 (Pin_3)
- net GND: now also J4.1 (Pin_1), J9.1 (Pin_1), U3.11 (GND), U4.11 (GND); no longer J4.4 (Pin_4), J9.4 (Pin_4)
- net at U5.2 (0_RX1_CRX2_CS1): now also U3.9 (A8)
- net at J5.3 (Pin_3), U5.25 (18_A4_SDA0): now also U4.7 (A6)
- net at J5.4 (Pin_4), U5.26 (19_A5_SCL0): now also U4.8 (A7)
- net at U5.3 (1_TX1_CTX2_MISO1): now also U3.8 (A7)
- net at U5.35 (24_A10_TX6_SCL2): now also J4.3 (Pin_3), U4.5 (A4); no longer J4.2 (Pin_2)
- net at U5.36 (25_A11_RX6_SDA2): now also J4.4 (Pin_4), U4.6 (A5); no longer J4.1 (Pin_1)
- net at U5.4 (2_OUT2): now also U3.7 (A6)
- net at U5.41 (30_CRX3): now also U4.4 (A3)
- net at J3.2 (Pin_2), U5.43 (32_OUT1B): now also U4.3 (A2)
- net at J3.1 (Pin_1), U5.44 (33_MCLK2): now also U4.1 (A1)
- net at U5.5 (3_LRCLK2): now also U3.6 (A5)
- net at U5.6 (4_BCLK2): now also U3.5 (A4)
- net at U5.7 (5_IN2): now also U3.4 (A3)
- net at J6.3 (Pin_3), U5.8 (6_OUT1D): now also U4.9 (A8)
- net at U5.9 (7_RX2_OUT1A): now also U3.3 (A2)
- net at J10.3 (Pin_3): now also U4.14 (B6)
- net at J10.4 (Pin_4): now also U4.13 (B7)
- net at M1.4 (A): now also U3.12 (B8)
- net at M1.3 (B): now also U3.13 (B7)
- net at M2.4 (A): now also U3.14 (B6)
- net at M2.3 (B): now also U3.15 (B5)
- net at M3.4 (A): now also U3.16 (B4)
- net at M3.3 (B): now also U3.17 (B3)
- net at M4.4 (A): now also U3.18 (B2)
- net at J11.3 (Pin_3): now also U4.12 (B8)
- net at M4.3 (B): now also U4.17 (B3)
- net at J8.1 (Pin_1): now also U4.20 (B1)
- net at J8.2 (Pin_2): now also U4.18 (B2)
- new net: J9.3 (Pin_3), U4.16 (B4)
- new net: J9.4 (Pin_4), U4.15 (B5)
Other:
- moved on the sheet: C10, C2, C5, C6, C7, C8, J8, J9, R1
